File: cc3000-ft232h.kicad_pcb (KiCad board)
At the start: 2 copper layers, 50 x 50 mm, 58 parts, among them CON1 USB-MINI-B, IC1 V_REG_LM1117SOT223, P1 CONN_4X2, P2 CONN_8, P3 CONN_13, P4 CONN_13, P5 CONN_4, P7 CONN_6, Q1 BCX51, Q2 BCX51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

Commit message: ftdi pronto(versao beta) + breakout
Parts:
- added C17: 0.1, SM0805, B.Cu at (168.8, 76.7)
- added P8: CONN_8, 1X08_LOCK, F.Cu at (126.4, 71.5)
- added P9: CONN_8, 1X08_LOCK, F.Cu at (126.4, 84.2)
- moved C11 3.40 mm to (169.3, 96.9)
- moved R1 3.40 mm to (167.5, 96.9)
- moved C15 1.50 mm to (165.7, 98.8)
- moved C16 1.50 mm to (164.0, 98.8)
Routing:
- net GND: track 350.6 -> 410.2 mm, vias 48 -> 54
- net /ft232h/VCC3V3: track 48.8 -> 66.3 mm, vias 2 -> 4
- net /ft232h/ACBUS9: track 0.00 -> 13.8 mm
- net /ft232h/ACBUS8: track 0.00 -> 12.2 mm
- net /ft232h/ACBUS7: track 0.00 -> 11.4 mm
- net /ft232h/ACBUS6: track 0.00 -> 9.96 mm
- net +3.3V: track 160.5 -> 167.8 mm
- net /ft232h/ACBUS4: track 20.0 -> 18.8 mm
- net /ft232h/VREGIN: track 21.0 -> 20.1 mm
- net /ft232h/ACBUS3: track 16.0 -> 15.4 mm

Commit message: ftdi pronto(versao beta) + breakout
Parts:
- removed FB4, FB5: FILTER, SM0805
- added P6: CONN_1, 1PIN_SMD, F.Cu at (169.3, 99.5)
- P7: footprint 1X06_LOCK -> 1X01
Connections:
- JP1 pad 2: N-0000066 -> N-0000040
- P5 pad 2: N-0000066 -> N-0000040
- U3 pad 6: /ft232h/D- -> /ft232h/USB_D-
- U3 pad 7: /ft232h/D+ -> /ft232h/USB_D+
Routing:
- net /ft232h/USB_D+: track 16.7 -> 26.2 mm
- net /ft232h/USB_D-: track 15.9 -> 24.4 mm
- net N-0000066: track 7.94 -> 0.00 mm
- net N-0000040: track 0.00 -> 7.94 mm
- net /ft232h/D+: track 7.56 -> 0.00 mm
- net /ft232h/D-: track 6.65 -> 0.00 mm
- net N-0000029: track 6.63 -> 8.60 mm

Commit message: ftdi pronto(versao beta) + breakout
Parts:
- P7: footprint 1X01 -> 1X06_LOCK
- moved P7 0.10 mm to (155.2, 117.9)
Changed lines of the file:
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@@
 (kicad_pcb (version 3) (host pcbnew "(2013-04-19 BZR 4011)-stable")
   (general
-    (links 191)
+    (links 196)
     (no_connects 1)
     (area 124.949999 69.949999 175.050001 120.050001)
@@
     (mod_text_width 0.15)
     (pad_size 1.5 1.5)
-    (pad_drill 0)
+    (pad_drill 0.6)
     (pad_to_mask_clearance 0)
     (aux_axis_origin 0 0)
@@
     )
   )
-  (module 1X01 (layer F.Cu)
-    (at 155.3 117.9)
-    (fp_text reference P7 (at 3.7338 -1.1938) (layer Eco1.User)
+  (module 1X06_LOCK (layer F.Cu)
+    (at 155.2 117.9)
+    (descr "This footprint was designed to help hold the alignment of a through-hole component (i.e.  6-pin header) while soldering it into place.")
+    (fp_text reference P7 (at 1.27 -1.143) (layer Eco1.User)
       (effects (font (size 1.27 1.27) (thickness 0.1016)))
     )
-    (fp_text value CONN_6 (at 2.54 3.81) (layer Eco1.User)
+    (fp_text value CONN_6 (at 2.54 3.937) (layer Eco1.User)
       (effects (font (size 1.27 1.27) (thickness 0.1016)))
     )
-    (fp_line (start 1.27 -0.635) (end 0.635 -1.27) (layer F.SilkS) (width 0.2032))
-    (fp_line (start 0.635 -1.27) (end -0.635 -1.27) (layer F.SilkS) (width 0.2032))
-    (fp_line (start -0.635 -1.27) (end -1.27 -0.635) (layer F.SilkS) (width 0.2032))
-    (fp_line (start -1.27 -0.635) (end -1.27 0.635) (layer F.SilkS) (width 0.2032))
-    (fp_line (start -1.27 0.635) (end -0.635 1.27) (layer F.SilkS) (width 0.2032))
-    (fp_line (start -0.635 1.27) (end 0.635 1.27) (layer F.SilkS) (width 0.2032))
-    (fp_line (start 0.635 1.27) (end 1.27 0.635) (layer F.SilkS) (width 0.2032))
-    (fp_line (start 1.27 0.635) (end 1.27 -0.635) (layer F.SilkS) (width 0.2032))
-    (fp_line (start -0.254 0.254) (end 0.254 0.254) (layer Cmts.User) (width 0.127))
-    (fp_line (start 0.254 0.254) (end 0.254 -0.254) (layer Cmts.User) (width 0.127))
-    (fp_line (start 0.254 -0.254) (end -0.254 -0.254) (layer Cmts.User) (width 0.127))
-    (fp_line (start -0.254 -0.254) (end -0.254 0.254) (layer Cmts.User) (width 0.127))
-    (pad 1 thru_hole oval (at 0 0 90) (size 1.8796 1.8796) (drill 1.016)
+    (fp_line (start -1.27 -0.508) (end -0.635 -1.143) (layer F.SilkS) (width 0.2032))
+    (fp_line (start -0.635 -1.143) (end 0.635 -1.143) (layer F.SilkS) (width 0.2032))
+    (fp_line (start 0.635 -1.143) (end 1.27 -0.508) (layer F.SilkS) (width 0.2032))
+    (fp_line (start 1.27 -0.508) (end 1.905 -1.143) (layer F.SilkS) (width 0.2032))
+    (fp_line (start 1.905 -1.143) (end 3.175 -1.143) (layer F.SilkS) (width 0.2032))
+    (fp_line (start 3.175 -1.143) (end 3.81 -0.508) (layer F.SilkS) (width 0.2032))
+    (fp_line (start 3.81 -0.508) (end 4.445 -1.143) (layer F.SilkS) (width 0.2032))
+    (fp_line (start 4.445 -1.143) (end 5.715 -1.143) (layer F.SilkS) (width 0.2032))
+    (fp_line (start 5.715 -1.143) (end 6.35 -0.508) (layer F.SilkS) (width 0.2032))
+    (fp_line (start 6.35 -0.508) (end 6.985 -1.143) (layer F.SilkS) (width 0.2032))
+    (fp_line (start 6.985 -1.143) (end 8.255 -1.143) (layer F.SilkS) (width 0.2032))
+    (fp_line (start 8.255 -1.143) (end 8.89 -0.508) (layer F.SilkS) (width 0.2032))
+    (fp_line (start 8.89 -0.508) (end 9.525 -1.143) (layer F.SilkS) (width 0.2032))
+    (fp_line (start 9.525 -1.143) (end 10.795 -1.143) (layer F.SilkS) (width 0.2032))
+    (fp_line (start 10.795 -1.143) (end 11.43 -0.508) (layer F.SilkS) (width 0.2032))
+    (fp_line (start 11.43 -0.508) (end 12.065 -1.143) (layer F.SilkS) (width 0.2032))
+    (fp_line (start 12.065 -1.143) (end 13.335 -1.143) (layer F.SilkS) (width 0.2032))
+    (fp_line (start 13.335 -1.143) (end 13.97 -0.508) (layer F.SilkS) (width 0.2032))
+    (fp_line (start 13.97 -0.508) (end 13.97 0.762) (layer F.SilkS) (width 0.2032))
+    (fp_line (start 13.97 0.762) (end 13.335 1.397) (layer F.SilkS) (width 0.2032))
+    (fp_line (start 13.335 1.397) (end 12.065 1.397) (layer F.SilkS) (width 0.2032))
+    (fp_line (start 12.065 1.397) (end 11.43 0.762) (layer F.SilkS) (width 0.2032))
+    (fp_line (start 11.43 0.762) (end 10.795 1.397) (layer F.SilkS) (width 0.2032))
+    (fp_line (start 10.795 1.397) (end 9.525 1.397) (layer F.SilkS) (width 0.2032))
+    (fp_line (start 9.525 1.397) (end 8.89 0.762) (layer F.SilkS) (width 0.2032))
+    (fp_line (start 8.89 0.762) (end 8.255 1.397) (layer F.SilkS) (width 0.2032))
+    (fp_line (start 8.255 1.397) (end 6.985 1.397) (layer F.SilkS) (width 0.2032))
+    (fp_line (start 6.985 1.397) (end 6.35 0.762) (layer F.SilkS) (width 0.2032))
+    (fp_line (start 6.35 0.762) (end 5.715 1.397) (layer F.SilkS) (width 0.2032))
+    (fp_line (start 5.715 1.397) (end 4.445 1.397) (layer F.SilkS) (width 0.2032))
+    (fp_line (start 4.445 1.397) (end 3.81 0.762) (layer F.SilkS) (width 0.2032))
+    (fp_line (start 3.81 0.762) (end 3.175 1.397) (layer F.SilkS) (width 0.2032))
+    (fp_line (start 3.175 1.397) (end 1.905 1.397) (layer F.SilkS) (width 0.2032))
+    (fp_line (start 1.905 1.397) (end 1.27 0.762) (layer F.SilkS) (width 0.2032))
+    (fp_line (start 1.27 0.762) (end 0.635 1.397) (layer F.SilkS) (width 0.2032))
+    (fp_line (start 0.635 1.397) (end -0.635 1.397) (layer F.SilkS) (width 0.2032))
+    (fp_line (start -0.635 1.397) (end -1.27 0.762) (layer F.SilkS) (width 0.2032))
+    (fp_line (start -1.27 0.762) (end -1.27 -0.508) (layer F.SilkS) (width 0.2032))
+    (fp_line (start 1.27 -0.508) (end 1.27 0.762) (layer F.SilkS) (width 0.2032))
+    (fp_line (start 3.81 -0.508) (end 3.81 0.762) (layer F.SilkS) (width 0.2032))
+    (fp_line (start 6.35 -0.508) (end 6.35 0.762) (layer F.SilkS) (width 0.2032))
+    (fp_line (start 8.89 -0.508) (end 8.89 0.762) (layer F.SilkS) (width 0.2032))
+    (fp_line (start 11.43 -0.508) (end 11.43 0.762) (layer F.SilkS) (width 0.2032))
+    (fp_line (start -0.2921 0.4191) (end 0.2921 0.4191) (layer Cmts.User) (width 0.127))
+    (fp_line (start 0.2921 0.4191) (end 0.2921 -0.1651) (layer Cmts.User) (width 0.127))
+    (fp_line (start 0.2921 -0.1651) (end -0.2921 -0.1651) (layer Cmts.User) (width 0.127))
+    (fp_line (start -0.2921 -0.1651) (end -0.2921 0.4191) (layer Cmts.User) (width 0.127))
+    (fp_line (start 2.2479 0.4191) (end 2.8321 0.4191) (layer Cmts.User) (width 0.127))
+    (fp_line (start 2.8321 0.4191) (end 2.8321 -0.1651) (layer Cmts.User) (width 0.127))
+    (fp_line (start 2.8321 -0.1651) (end 2.2479 -0.1651) (layer Cmts.User) (width 0.127))
+    (fp_line (start 2.2479 -0.1651) (end 2.2479 0.4191) (layer Cmts.User) (width 0.127))
+    (fp_line (start 4.7879 0.4191) (end 5.3721 0.4191) (layer Cmts.User) (width 0.127))
+    (fp_line (start 5.3721 0.4191) (end 5.3721 -0.1651) (layer Cmts.User) (width 0.127))
+    (fp_line (start 5.3721 -0.1651) (end 4.7879 -0.1651) (layer Cmts.User) (width 0.127))
+    (fp_line (start 4.7879 -0.1651) (end 4.7879 0.4191) (layer Cmts.User) (width 0.127))
+    (fp_line (start 7.3279 0.4191) (end 7.9121 0.4191) (layer Cmts.User) (width 0.127))
+    (fp_line (start 7.9121 0.4191) (end 7.9121 -0.1651) (layer Cmts.User) (width 0.127))
+    (fp_line (start 7.9121 -0.1651) (end 7.3279 -0.1651) (layer Cmts.User) (width 0.127))
+    (fp_line (start 7.3279 -0.1651) (end 7.3279 0.4191) (layer Cmts.User) (width 0.127))
+    (fp_line (start 9.8679 0.4191) (end 10.4521 0.4191) (layer Cmts.User) (width 0.127))
+    (fp_line (start 10.4521 0.4191) (end 10.4521 -0.1651) (layer Cmts.User) (width 0.127))
+    (fp_line (start 10.4521 -0.1651) (end 9.8679 -0.1651) (layer Cmts.User) (width 0.127))
+    (fp_line (start 9.8679 -0.1651) (end 9.8679 0.4191) (layer Cmts.User) (width 0.127))
+    (fp_line (start 12.4079 0.4191) (end 12.9921 0.4191) (layer Cmts.User) (width 0.127))
+    (fp_line (start 12.9921 0.4191) (end 12.9921 -0.1651) (layer Cmts.User) (width 0.127))
+    (fp_line (start 12.9921 -0.1651) (end 12.4079 -0.1651) (layer Cmts.User) (width 0.127))
+    (fp_line (start 12.4079 -0.1651) (end 12.4079 0.4191) (layer Cmts.User) (width 0.127))
+    (pad 1 thru_hole oval (at 0 0) (size 1.8796 1.8796) (drill 1.016)
       (layers *.Cu *.Mask)
       (net 38 GND)
     )
+    (pad 2 thru_hole oval (at 2.54 0.254) (size 1.8796 1.8796) (drill 1.016)
+      (layers *.Cu *.Mask)
+      (net 55 N-0000040)
+    )
+    (pad 3 thru_hole oval (at 5.08 0) (size 1.8796 1.8796) (drill 1.016)
+      (layers *.Cu *.Mask)
+      (net 22 /ft232h/ADBUS1)
+    )
+    (pad 4 thru_hole oval (at 7.62 0.254) (size 1.8796 1.8796) (drill 1.016)
+      (layers *.Cu *.Mask)
+      (net 21 /ft232h/ADBUS0)
+    )
+    (pad 5 thru_hole oval (at 10.16 0) (size 1.8796 1.8796) (drill 1.016)
+      (layers *.Cu *.Mask)
+      (net 23 /ft232h/ADBUS2)
+    )
+    (pad 6 thru_hole oval (at 12.7 0.254) (size 1.8796 1.8796) (drill 1.016)
+      (layers *.Cu *.Mask)
+      (net 24 /ft232h/ADBUS3)
+    )
   )
   (dimension 21.336 (width 0.3) (layer Dwgs.User)
@@
   (segment (start 167.44886 83.2) (end 167.14958 83.2) (width 0.254) (layer F.Cu) (net 48))
   (segment (start 167.14958 83.2) (end 163.94958 86.4) (width 0.254) (layer F.Cu) (net 48))
-  (segment (start 169.3 99.5) (end 167.4 99.5) (width 0.33) (layer F.Cu) (net 49) (status 400000))
+  (segment (start 169.3 99.5) (end 167.4 99.5) (width 0.33) (layer F.Cu) (net 49))
   (segment (start 167.4 99.5) (end 167.35 99.45) (width 0.33) (layer F.Cu) (net 49))
   (segment (start 167.5 97.8525) (end 167.5 99.3) (width 0.254) (layer B.Cu) (net 49))

Commit message: ftdi done + breakout done
Parts:
- added ??1: 74LVC138AD, SO16N, F.Cu at (135.3, 77.8)
- added U4: 74LVC138AD, SparkFun-TSSOP16, B.Cu at (135.2, 77.7)
Connections:
- P8 pad 1: (no net) -> N-0000071
- P8 pad 2: (no net) -> N-0000072
- P8 pad 3: (no net) -> N-0000070
- P8 pad 4: (no net) -> N-0000079
- P8 pad 5: (no net) -> N-0000080
- P8 pad 6: (no net) -> N-0000081
- P8 pad 7: (no net) -> N-0000082
- P8 pad 8: (no net) -> N-0000083
- P9 pad 1: (no net) -> N-0000073
- P9 pad 2: (no net) -> N-0000078
- P9 pad 3: (no net) -> N-0000077
- P9 pad 4: (no net) -> N-0000076
- P9 pad 5: (no net) -> N-0000075
- P9 pad 6: (no net) -> N-0000074
- P9 pad 7: (no net) -> N-0000068
- P9 pad 8: (no net) -> N-0000069
Routing:
- net N-0000069: track 0.00 -> 13.9 mm
- net N-0000071: track 0.00 -> 13.9 mm
- net N-0000083: track 0.00 -> 13.7 mm
- net N-0000073: track 0.00 -> 13.7 mm
- net N-0000082: track 0.00 -> 11.8 mm
- net N-0000078: track 0.00 -> 11.4 mm
- net N-0000072: track 0.00 -> 11.4 mm
- net N-0000068: track 0.00 -> 11.3 mm
- net N-0000074: track 0.00 -> 9.14 mm
- net N-0000070: track 0.00 -> 9.07 mm
- net N-0000081: track 0.00 -> 8.78 mm
- net N-0000077: track 0.00 -> 8.65 mm
- net N-0000080: track 0.00 -> 7.50 mm
- net N-0000076: track 0.00 -> 7.47 mm
- net N-0000075: track 0.00 -> 6.99 mm
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
Commit message: ftdi done + breakout done + silk done
Parts:
- added C18: 10u, SM0805, B.Cu at (154.7, 73.5)
- added C19: 10u, SM0805, B.Cu at (149.0, 80.1)
- C8, C9: moved to B.Cu
- moved D2 0.50 mm to (169.3, 103.5)
- moved D1 0.40 mm to (169.3, 106.7)
- moved C9 0.10 mm to (170.5, 91.6)
Routing:
- net GND: track 410.2 -> 422.6 mm, vias 54 -> 55
- net (no net): track 0.00 -> 2.21 mm
- net N-0000027: track 1.62 -> 3.80 mm, vias 0 -> 1
- net +5V: track 55.7 -> 57.2 mm
- net /ft232h/VCC3V3: track 66.3 -> 65.4 mm
- net +3.3V: track 167.8 -> 168.5 mm
- net N-0000036: track 2.54 -> 1.77 mm
- net N-0000037: track 2.63 -> 2.01 mm
- net /ft232h/VCORE: track 5.89 -> 5.93 mm, vias 0 -> 1
- net N-0000032: track 6.84 -> 6.80 mm, vias 0 -> 1
Other:
- board text added: "3V3 O/F"
- board text added: "5V"
- board text added: "AC0"
- board text added: "AC1"
- board text added: "AC2"
- board text added: "AC3"
- board text added: "AC4"
- board text added: "AC5"
- board text added: "AC6"
- board text added: "AC7"
- board text added: "AC8"
- board text added: "AC9"
- board text added: "AD0"
- board text added: "AD1"
- board text added: "AD2"
- board text added: "AD3"
- board text added: "AD4"
- board text added: "AD5"
- board text added: "AD6"
- board text added: "AD7"
- board text added: "DI"
- board text added: "DO"
- board text added: "POWER LED"
- board text added: "Pull-up"
- board text added: "RX"
- board text added: "RXD TDI SDA MOSI"
- board text added: "SCL"
- board text added: "SCL SCKL"
- board text added: "SDA"
- board text added: "TCK AD0"
- board text added: "TDO MISO AD2"
- board text added: "TMS CS AD3"
- board text added: "TX"
- board text added: "TXD"

Commit message: git link
Routing:
- net /ft232h/ADBUS7: track 15.7 -> 14.9 mm
- net (no net): track 2.21 -> 2.93 mm, vias 0 -> 1
- net /ft232h/USB_D+: track 26.2 -> 25.6 mm
Other:
- board text added: "3V3 Trgt"
- board text added: "Rev. 1"
- board text added: "https://github.com/ brNX/cc3000-ft232h4"
- board text removed: "3V3 O/F"
