File: cc3000.sch (KiCad schematic (older format))
At the start: 8 parts, among them P1 CONN_4X2, P2 CONN_8, U1 U.FL_U.FL, U2 CC3000TEXAS_CC3000

Commit message: most erc errors fixed
Changed lines of the file:
@@
-EESchema Schematic File Version 2  date 03-08-2013 18:53:09
+EESchema Schematic File Version 2
 LIBS:power
 LIBS:device
@@
 $EndComp
 $Comp
-L PWR_FLAG #FLG015
-U 1 1 51E58D36
-P 6300 2000
-F 0 "#FLG015" H 6300 2095 30  0001 C CNN
-F 1 "PWR_FLAG" H 6300 2180 30  0000 C CNN
-F 2 "" H 6300 2000 60  0000 C CNN
-F 3 "" H 6300 2000 60  0000 C CNN
-	1    6300 2000
-	1    0    0    -1
-$EndComp
-$Comp
-L GND #PWR016
+L GND #PWR015
 U 1 1 51E58D3C
 P 6000 2150
-F 0 "#PWR016" H 6000 2150 30  0001 C CNN
+F 0 "#PWR015" H 6000 2150 30  0001 C CNN
 F 1 "GND" H 6000 2080 30  0001 C CNN
 F 2 "" H 6000 2150 60  0000 C CNN
@@
 	1    0    0    -1
 $EndComp
-$Comp
-L +3,3V #PWR017
-U 1 1 51E58D42
-P 6300 2150
-F 0 "#PWR017" H 6300 2110 30  0001 C CNN
-F 1 "+3,3V" H 6300 2260 30  0000 C CNN
-F 2 "" H 6300 2150 60  0000 C CNN
-F 3 "" H 6300 2150 60  0000 C CNN
-	1    6300 2150
-	-1   0    0    1
-$EndComp
 Wire Wire Line
 	6000 2000 6000 2150
-Wire Wire Line
-	6300 2000 6300 2150
 $Comp
 L C C2
@@
 $EndComp
 $Comp
-L +3,3V #PWR018
+L +3,3V #PWR016
 U 1 1 51E599B8
 P 7300 4500
-F 0 "#PWR018" H 7300 4460 30  0001 C CNN
+F 0 "#PWR016" H 7300 4460 30  0001 C CNN
 F 1 "+3,3V" H 7300 4610 30  0000 C CNN
 F 2 "" H 7300 4500 60  0000 C CNN
@@
 $EndComp
 $Comp
-L +3,3V #PWR019
+L +3,3V #PWR017
 U 1 1 51E599BE
 P 7650 4500
-F 0 "#PWR019" H 7650 4460 30  0001 C CNN
+F 0 "#PWR017" H 7650 4460 30  0001 C CNN
 F 1 "+3,3V" H 7650 4610 30  0000 C CNN
 F 2 "" H 7650 4500 60  0000 C CNN
@@
 $EndComp
 $Comp
-L GND #PWR020
+L GND #PWR018
 U 1 1 51E599C4
 P 7300 4900
-F 0 "#PWR020" H 7300 4900 30  0001 C CNN
+F 0 "#PWR018" H 7300 4900 30  0001 C CNN
 F 1 "GND" H 7300 4830 30  0001 C CNN
 F 2 "" H 7300 4900 60  0000 C CNN
@@
 $EndComp
 $Comp
-L GND #PWR021
+L GND #PWR019
 U 1 1 51E599D0
 P 7650 4900
-F 0 "#PWR021" H 7650 4900 30  0001 C CNN
+F 0 "#PWR019" H 7650 4900 30  0001 C CNN
 F 1 "GND" H 7650 4830 30  0001 C CNN
 F 2 "" H 7650 4900 60  0000 C CNN
@@
 $EndComp
 $Comp
-L +3,3V #PWR022
+L +3,3V #PWR020
 U 1 1 51E59BA0
 P 7950 4500
-F 0 "#PWR022" H 7950 4460 30  0001 C CNN
+F 0 "#PWR020" H 7950 4460 30  0001 C CNN
 F 1 "+3,3V" H 7950 4610 30  0000 C CNN
 F 2 "" H 7950 4500 60  0000 C CNN
@@
 $EndComp
 $Comp
-L GND #PWR023
+L GND #PWR021
 U 1 1 51E59BA6
 P 7950 4900
-F 0 "#PWR023" H 7950 4900 30  0001 C CNN
+F 0 "#PWR021" H 7950 4900 30  0001 C CNN
 F 1 "GND" H 7950 4830 30  0001 C CNN
 F 2 "" H 7950 4900 60  0000 C CNN
@@
 $EndComp
 $Comp
-L +3,3V #PWR024
+L +3,3V #PWR022
 U 1 1 51E9E8F9
 P 9400 3350
-F 0 "#PWR024" H 9400 3310 30  0001 C CNN
+F 0 "#PWR022" H 9400 3310 30  0001 C CNN
 F 1 "+3,3V" H 9400 3460 30  0000 C CNN
 F 2 "" H 9400 3350 60  0000 C CNN
@@
 $EndComp
 $Comp
-L GND #PWR025
+L GND #PWR023
 U 1 1 51E9E8FF
 P 9400 3450
-F 0 "#PWR025" H 9400 3450 30  0001 C CNN
+F 0 "#PWR023" H 9400 3450 30  0001 C CNN
 F 1 "GND" H 9400 3380 30  0001 C CNN
 F 2 "" H 9400 3450 60  0000 C CNN
