File: ft232h.sch (KiCad schematic (older format))
At the start: 50 parts, among them CON1 USB-MINI-B, IC1 V_REG_LM1117SOT223, P3 CONN_13, P4 CONN_13, P5 CONN_4, P6 CONN_1, P7 CONN_6, Q1 BCX51, Q2 BCX51, U3 FT232H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

Commit message: ftdi done + breakout done + silk done
Parts:
- added C18, C19: 10u, ~, symbol C

Commit message: decoupling caps , silk screen modified
Parts:
- added C20, C21, C22: 0.1, ~, symbol C
- R1: value 12K -> 10k
Connections:
- wire segments 132 -> 136
Changed lines of the file:
@@
-EESchema Schematic File Version 2  date 03-08-2013 22:48:25
+EESchema Schematic File Version 2
 LIBS:power
 LIBS:device
@@
 LIBS:sn74cb3t3245
 LIBS:cc3000-ft232h-cache
-EELAYER 27 0
+EELAYER 24 0
 EELAYER END
 $Descr A4 11693 8268
@@
 P 3950 4150
 F 0 "R1" V 4030 4150 40  0000 C CNN
-F 1 "12K" V 3957 4151 40  0000 C CNN
+F 1 "10k" V 3957 4151 40  0000 C CNN
 F 2 "~" V 3880 4150 30  0000 C CNN
 F 3 "~" H 3950 4150 30  0000 C CNN
@@
 VREGIN
 $Comp
-L +3.3V #PWR59
+L +3.3V #PWR60
 U 1 1 51FB6478
 P 9000 4350
-F 0 "#PWR59" H 9000 4310 30  0001 C CNN
+F 0 "#PWR60" H 9000 4310 30  0001 C CNN
 F 1 "+3.3V" H 9000 4460 30  0000 C CNN
 F 2 "" H 9000 4350 60  0000 C CNN
@@
 $EndComp
 $Comp
-L +3.3V #PWR58
+L +3.3V #PWR59
 U 1 1 51FB6850
 P 8400 3550
-F 0 "#PWR58" H 8400 3510 30  0001 C CNN
+F 0 "#PWR59" H 8400 3510 30  0001 C CNN
 F 1 "+3.3V" H 8400 3660 30  0000 C CNN
 F 2 "" H 8400 3550 60  0000 C CNN
@@
 	1    0    0    -1
 $EndComp
+$Comp
+L C C18
+U 1 1 51FD7A84
+P 850 1050
+F 0 "C18" H 850 1150 40  0000 L CNN
+F 1 "10u" H 856 965 40  0000 L CNN
+F 2 "~" H 888 900 30  0000 C CNN
+F 3 "~" H 850 1050 60  0000 C CNN
+	1    850  1050
+	1    0    0    -1
+$EndComp
+$Comp
+L C C19
+U 1 1 51FD7A8B
+P 1650 1350
+F 0 "C19" H 1650 1450 40  0000 L CNN
+F 1 "10u" H 1656 1265 40  0000 L CNN
+F 2 "~" H 1688 1200 30  0000 C CNN
+F 3 "~" H 1650 1350 60  0000 C CNN
+	1    1650 1350
+	1    0    0    -1
+$EndComp
+$Comp
+L GND #PWR33
+U 1 1 51FD7A91
+P 1650 1550
+F 0 "#PWR33" H 1650 1550 30  0001 C CNN
+F 1 "GND" H 1650 1480 30  0001 C CNN
+F 2 "" H 1650 1550 60  0000 C CNN
+F 3 "" H 1650 1550 60  0000 C CNN
+	1    1650 1550
+	1    0    0    -1
+$EndComp
+$Comp
+L GND #PWR26
+U 1 1 51FD7A97
+P 850 1250
+F 0 "#PWR26" H 850 1250 30  0001 C CNN
+F 1 "GND" H 850 1180 30  0001 C CNN
+F 2 "" H 850 1250 60  0000 C CNN
+F 3 "" H 850 1250 60  0000 C CNN
+	1    850  1250
+	1    0    0    -1
+$EndComp
+$Comp
+L C C21
+U 1 1 520CEA32
+P 6050 1900
+F 0 "C21" H 6050 2000 40  0000 L CNN
+F 1 "0.1" H 6056 1815 40  0000 L CNN
+F 2 "~" H 6088 1750 30  0000 C CNN
+F 3 "~" H 6050 1900 60  0000 C CNN
+	1    6050 1900
+	0    -1   -1   0
+$EndComp
+$Comp
+L C C22
+U 1 1 520CEA3B
+P 6150 2100
+F 0 "C22" H 6150 2200 40  0000 L CNN
+F 1 "0.1" H 6156 2015 40  0000 L CNN
+F 2 "~" H 6188 1950 30  0000 C CNN
+F 3 "~" H 6150 2100 60  0000 C CNN
+	1    6150 2100
+	0    -1   -1   0
+$EndComp
+$Comp
+L C C20
+U 1 1 520CEA41
+P 5950 1700
+F 0 "C20" H 5950 1800 40  0000 L CNN
+F 1 "0.1" H 5956 1615 40  0000 L CNN
+F 2 "~" H 5988 1550 30  0000 C CNN
+F 3 "~" H 5950 1700 60  0000 C CNN
+	1    5950 1700
+	0    -1   -1   0
+$EndComp
 Wire Wire Line
 	5250 5200 6250 5200
@@
 	4350 3500 4650 3500
 Wire Wire Line
-	5750 2400 6100 2400
-Connection ~ 5850 2400
-Wire Wire Line
 	3900 3300 3900 3200
 Wire Wire Line
@@
 Wire Wire Line
 	3500 3900 3950 3900
-Connection ~ 3500 3000
 Wire Wire Line
 	3950 5450 3950 5350
@@
 Wire Wire Line
 	3500 4600 3500 4750
-Connection ~ 10500 2750
-Connection ~ 9950 2850
-Connection ~ 9950 3050
-Connection ~ 9950 2950
 Wire Wire Line
 	9600 4250 9950 4250
@@
 	4200 3000 4650 3000
 Wire Wire Line
-	4200 3000 4200 2600
-Wire Wire Line
-	3500 2600 6100 2600
-Wire Wire Line
-	6100 2600 6100 2400
-Connection ~ 5950 2400
-Wire Wire Line
 	2800 1700 3250 1700
 Wire Wire Line
 	3950 1700 5650 1700
 Wire Wire Line
-	3100 2150 3100 1700
+	3100 1300 3100 2150
 Wire Wire Line
 	800  2500 1250 2500
@@
 Connection ~ 3100 1700
 Wire Wire Line
-	3500 2600 3500 3900
-Connection ~ 4200 2600
-Wire Wire Line
 	3650 6300 4000 6300
 Wire Wire Line
@@
 Wire Wire Line
 	9600 4300 9600 4350
-Connection ~ 9500 3600
 Wire Wire Line
 	9150 3050 10500 3050
@@
 	1450 950  1650 950
 Connection ~ 1650 950
-$Comp
-L C C18
-U 1 1 51FD7A84
-P 850 1050
-F 0 "C18" H 850 1150 40  0000 L CNN
-F 1 "10u" H 856 965 40  0000 L CNN
-F 2 "~" H 888 900 30  0000 C CNN
-F 3 "~" H 850 1050 60  0000 C CNN
-	1    850  1050
-	1    0    0    -1
-$EndComp
-$Comp
-L C C19
-U 1 1 51FD7A8B
-P 1650 1350
-F 0 "C19" H 1650 1450 40  0000 L CNN
-F 1 "10u" H 1656 1265 40  0000 L CNN
-F 2 "~" H 1688 1200 30  0000 C CNN
-F 3 "~" H 1650 1350 60  0000 C CNN
-	1    1650 1350
-	1    0    0    -1
-$EndComp
-$Comp
-L GND #PWR33
-U 1 1 51FD7A91
-P 1650 1550
-F 0 "#PWR33" H 1650 1550 30  0001 C CNN
-F 1 "GND" H 1650 1480 30  0001 C CNN
-F 2 "" H 1650 1550 60  0000 C CNN
-F 3 "" H 1650 1550 60  0000 C CNN
-	1    1650 1550
-	1    0    0    -1
-$EndComp
-$Comp
-L GND #PWR26
-U 1 1 51FD7A97
-P 850 1250
-F 0 "#PWR26" H 850 1250 30  0001 C CNN
-F 1 "GND" H 850 1180 30  0001 C CNN
-F 2 "" H 850 1250 60  0000 C CNN
-F 3 "" H 850 1250 60  0000 C CNN
-	1    850  1250
-	1    0    0    -1
-$EndComp
+Wire Wire Line
+	3100 1300 5750 1300
+Wire Wire Line
+	5750 1300 5750 2400
+Connection ~ 5750 1700
+Wire Wire Line
+	5850 1900 5750 1900
+Connection ~ 5750 1900
+Wire Wire Line
+	5750 2100 5950 2100
+Connection ~ 5750 2100
+Wire Wire Line
+	5850 2400 5850 1900
+Wire Wire Line
+	5950 2100 5950 2400
+$Comp
+L GND #PWR58
+U 1 1 520CF27C
+P 6500 1900
+F 0 "#PWR58" H 6500 1900 30  0001 C CNN
+F 1 "GND" H 6500 1830 30  0001 C CNN
+F 2 "" H 6500 1900 60  0000 C CNN
+F 3 "" H 6500 1900 60  0000 C CNN
+	1    6500 1900
+	0    -1   -1   0
+$EndComp
+Wire Wire Line
+	6350 1700 6350 2100
+Wire Wire Line
+	6350 1700 6150 1700
+Wire Wire Line
+	6250 1900 6500 1900
+Connection ~ 6350 1900
+Text Label 3500 3900 2    60   ~ 0
+VCC3V3
 $EndSCHEMATC
